File: sensors/Rasp_pi.kicad_sch (KiCad schematic)
At the start: 1 part

Commit message: Version 2022.09.20 - Added Terminal Blocks
Parts:
- J?: footprint (none) -> Connector_PinHeader_2.54mm:PinHeader_2x20_P2.54mm_Vertical
Changed lines of the file:
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@@
       (effects (font (size 1.27 1.27)) (justify left))
     )
-    (property "Footprint" "" (id 2) (at 152.4 98.425 0)
+    (property "Footprint" "Connector_PinHeader_2.54mm:PinHeader_2x20_P2.54mm_Vertical" (id 2) (at 152.4 98.425 0)
       (effects (font (size 1.27 1.27)) hide)
     )
